File: MainPCB/PicoLX.kicad_sch (KiCad schematic)
At the start: 83 parts, among them J1 USB_C_Receptacle_USB2.0, SW1 SW_Push, SW1 Test, SW2 Service, U1 RP2040, U2 W25Q32JVSS, U3 NCP1117-3.3_SOT223, U4 SN74LV1T34DBV, Y1 12.000MHz

Commit message: Fixed minor switch alignment issues (<0.05mm)
Parts:
- C18, C19, C20, C21, C22, C23, C24, C25, C26, C27, C28, C29, C30, C31, C32, C33, C34, C35, C36: LCSC C15008 -> C437555
Changed lines of the file:
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@@
       (effects (font (size 1.27 1.27)) hide)
     )
-    (property "LCSC" "C15008" (at 263.525 47.625 0)
+    (property "LCSC" "C437555" (at 263.525 47.625 0)
       (effects (font (size 1.27 1.27)) hide)
     )
@@
       (effects (font (size 1.27 1.27)) hide)
     )
-    (property "LCSC" "C15008" (at 251.46 133.35 0)
+    (property "LCSC" "C437555" (at 251.46 133.35 0)
       (effects (font (size 1.27 1.27)) hide)
     )
@@
       (effects (font (size 1.27 1.27)) hide)
     )
-    (property "LCSC" "C15008" (at 243.205 55.245 0)
+    (property "LCSC" "C437555" (at 243.205 55.245 0)
       (effects (font (size 1.27 1.27)) hide)
     )
@@
       (effects (font (size 1.27 1.27)) hide)
     )
-    (property "LCSC" "C15008" (at 251.46 16.51 0)
+    (property "LCSC" "C437555" (at 251.46 16.51 0)
       (effects (font (size 1.27 1.27)) hide)
     )
@@
       (effects (font (size 1.27 1.27)) hide)
     )
-    (property "LCSC" "C15008" (at 231.14 16.51 0)
+    (property "LCSC" "C437555" (at 231.14 16.51 0)
       (effects (font (size 1.27 1.27)) hide)
     )
@@
       (effects (font (size 1.27 1.27)) hide)
     )
-    (property "LCSC" "C15008" (at 233.045 47.625 0)
+    (property "LCSC" "C437555" (at 233.045 47.625 0)
       (effects (font (size 1.27 1.27)) hide)
     )
@@
       (effects (font (size 1.27 1.27)) hide)
     )
-    (property "LCSC" "C15008" (at 243.205 47.625 0)
+    (property "LCSC" "C437555" (at 243.205 47.625 0)
       (effects (font (size 1.27 1.27)) hide)
     )
@@
       (effects (font (size 1.27 1.27)) hide)
     )
-    (property "LCSC" "C15008" (at 222.885 47.625 0)
+    (property "LCSC" "C437555" (at 222.885 47.625 0)
       (effects (font (size 1.27 1.27)) hide)
     )
@@
       (effects (font (size 1.27 1.27)) hide)
     )
-    (property "LCSC" "C15008" (at 241.3 133.35 0)
+    (property "LCSC" "C437555" (at 241.3 133.35 0)
       (effects (font (size 1.27 1.27)) hide)
     )
@@
       (effects (font (size 1.27 1.27)) hide)
     )
-    (property "LCSC" "C15008" (at 233.045 55.245 0)
+    (property "LCSC" "C437555" (at 233.045 55.245 0)
       (effects (font (size 1.27 1.27)) hide)
     )
@@
       (effects (font (size 1.27 1.27)) hide)
     )
-    (property "LCSC" "C15008" (at 261.62 16.51 0)
+    (property "LCSC" "C437555" (at 261.62 16.51 0)
       (effects (font (size 1.27 1.27)) hide)
     )
@@
       (effects (font (size 1.27 1.27)) hide)
     )
-    (property "LCSC" "C15008" (at 210.82 16.51 0)
+    (property "LCSC" "C437555" (at 210.82 16.51 0)
       (effects (font (size 1.27 1.27)) hide)
     )
@@
       (effects (font (size 1.27 1.27)) hide)
     )
-    (property "LCSC" "C15008" (at 263.525 55.245 0)
+    (property "LCSC" "C437555" (at 263.525 55.245 0)
       (effects (font (size 1.27 1.27)) hide)
     )
@@
       (effects (font (size 1.27 1.27)) hide)
     )
-    (property "LCSC" "C15008" (at 231.14 133.35 0)
+    (property "LCSC" "C437555" (at 231.14 133.35 0)
       (effects (font (size 1.27 1.27)) hide)
     )
@@
       (effects (font (size 1.27 1.27)) hide)
     )
-    (property "LCSC" "C15008" (at 241.3 16.51 0)
+    (property "LCSC" "C437555" (at 241.3 16.51 0)
       (effects (font (size 1.27 1.27)) hide)
     )
@@
       (effects (font (size 1.27 1.27)) hide)
     )
-    (property "LCSC" "C15008" (at 220.98 16.51 0)
+    (property "LCSC" "C437555" (at 220.98 16.51 0)
       (effects (font (size 1.27 1.27)) hide)
     )
@@
       (effects (font (size 1.27 1.27)) hide)
     )
-    (property "LCSC" "C15008" (at 222.885 55.245 0)
+    (property "LCSC" "C437555" (at 222.885 55.245 0)
       (effects (font (size 1.27 1.27)) hide)
     )
@@
       (effects (font (size 1.27 1.27)) hide)
     )
-    (property "LCSC" "C15008" (at 253.365 55.245 0)
+    (property "LCSC" "C437555" (at 253.365 55.245 0)
       (effects (font (size 1.27 1.27)) hide)
     )
@@
       (effects (font (size 1.27 1.27)) hide)
     )
-    (property "LCSC" "C15008" (at 253.365 47.625 0)
-      (effects (font (size 1.27 1.27)) hide)
-    )
+    (property "LCSC" "C437555" (at 253.365 47.625 0)
+      (effects (font (size 1.27 1.27)) hide)
+    )
